Commit message: remove redundant links from ur3(e)

File: universal_robots/ros/ur3/ur3.urdf (robot description, URDF)
Before this commit: robot ur3_robot, 11 links, 10 joints
Links:
- removed link base
- removed link base_link_inertia
- removed link tool0
- link base_link: geometry visual mesh filename=meshes/base.dae
Joints:
- removed joint base_link-base_fixed_joint
- removed joint base_link-base_link_inertia
- removed joint flange-tool0
- joint shoulder_pan_joint: parent base_link_inertia -> base_link
- joint wrist_3-flange: origin xyz=0 0 0 rpy=0 -1.5707963267948966 -1.5707963267948966 -> (none)

File: universal_robots/ros/ur3e/ur3e.urdf (robot description, URDF)
Before this commit: robot ur3e_robot, 11 links, 10 joints
Links:
- removed link base
- removed link base_link_inertia
- removed link tool0
- link base_link: geometry visual mesh filename=meshes/base.dae
Joints:
- removed joint base_link-base_fixed_joint
- removed joint base_link-base_link_inertia
- removed joint flange-tool0
- joint shoulder_pan_joint: parent base_link_inertia -> base_link
- joint wrist_3-flange: origin xyz=0 0 0 rpy=0 -1.5707963267948966 -1.5707963267948966 -> (none)
