Commit message: remove redundant links from ur5/10(e)

File: universal_robots/ros/ur10/ur10.urdf (robot description, URDF)
Before this commit: robot ur10_robot, 11 links, 10 joints
Links:
- removed link base_link_inertia
- link base_link: geometry visual mesh filename=meshes/base.dae
Joints:
- removed joint base_link-base_link_inertia
- joint shoulder_pan_joint: parent base_link_inertia -> base_link

File: universal_robots/ros/ur10e/ur10e.urdf (robot description, URDF)
Before this commit: robot ur10e_robot, 11 links, 10 joints
Links:
- removed link base_link_inertia
- link base_link: geometry visual mesh filename=meshes/base.dae
Joints:
- removed joint base_link-base_link_inertia
- joint shoulder_pan_joint: parent base_link_inertia -> base_link

File: universal_robots/ros/ur5/ur5.urdf (robot description, URDF)
Before this commit: robot ur5_robot, 11 links, 10 joints
Links:
- removed link base_link_inertia
- link base_link: geometry visual mesh filename=meshes/base.dae
Joints:
- removed joint base_link-base_link_inertia
- joint shoulder_pan_joint: parent base_link_inertia -> base_link

File: universal_robots/ros/ur5e/ur5e.urdf (robot description, URDF)
Before this commit: robot ur5e_robot, 11 links, 10 joints
Links:
- removed link base_link_inertia
- link base_link: geometry visual mesh filename=meshes/base.dae
Joints:
- removed joint base_link-base_link_inertia
- joint shoulder_pan_joint: parent base_link_inertia -> base_link

Commit message: remove tool0 and base frame for now

File: universal_robots/ros/ur10/ur10.urdf (robot description, URDF)
Before this commit: robot ur10_robot, 10 links, 9 joints
Links:
- removed link base
- removed link tool0
Joints:
- removed joint base_link-base_fixed_joint
- removed joint flange-tool0
- joint wrist_3-flange: origin xyz=0 0 0 rpy=0 -1.5707963267948966 -1.5707963267948966 -> (none)

File: universal_robots/ros/ur10e/ur10e.urdf (robot description, URDF)
Before this commit: robot ur10e_robot, 10 links, 9 joints
Links:
- removed link base
- removed link tool0
Joints:
- removed joint base_link-base_fixed_joint
- removed joint flange-tool0
- joint wrist_3-flange: origin xyz=0 0 0 rpy=0 -1.5707963267948966 -1.5707963267948966 -> (none)

File: universal_robots/ros/ur5/ur5.urdf (robot description, URDF)
Before this commit: robot ur5_robot, 10 links, 9 joints
Links:
- removed link base
- removed link tool0
Joints:
- removed joint base_link-base_fixed_joint
- removed joint flange-tool0
- joint wrist_3-flange: origin xyz=0 0 0 rpy=0 -1.5707963267948966 -1.5707963267948966 -> (none)

File: universal_robots/ros/ur5e/ur5e.urdf (robot description, URDF)
Before this commit: robot ur5e_robot, 10 links, 9 joints
Links:
- removed link base
- removed link tool0
Joints:
- removed joint base_link-base_fixed_joint
- removed joint flange-tool0
- joint wrist_3-flange: origin xyz=0 0 0 rpy=0 -1.5707963267948966 -1.5707963267948966 -> (none)

Commit message: remove flange frame to avoid confusion with ROS

File: universal_robots/ros/ur10/ur10.urdf (robot description, URDF)
Before this commit: robot ur10_robot, 8 links, 7 joints
Links:
- removed link flange
Joints:
- removed joint wrist_3-flange

File: universal_robots/ros/ur10e/ur10e.urdf (robot description, URDF)
Before this commit: robot ur10e_robot, 8 links, 7 joints
Links:
- removed link flange
Joints:
- removed joint wrist_3-flange

File: universal_robots/ros/ur3/ur3.urdf (robot description, URDF)
Before this commit: robot ur3_robot, 8 links, 7 joints
Links:
- removed link flange
Joints:
- removed joint wrist_3-flange

File: universal_robots/ros/ur3e/ur3e.urdf (robot description, URDF)
Before this commit: robot ur3e_robot, 8 links, 7 joints
Links:
- removed link flange
Joints:
- removed joint wrist_3-flange

File: universal_robots/ros/ur5/ur5.urdf (robot description, URDF)
Before this commit: robot ur5_robot, 8 links, 7 joints
Links:
- removed link flange
Joints:
- removed joint wrist_3-flange

File: universal_robots/ros/ur5e/ur5e.urdf (robot description, URDF)
Before this commit: robot ur5e_robot, 8 links, 7 joints
Links:
- removed link flange
Joints:
- removed joint wrist_3-flange
